File: circuit/GoWin Electrical.sch (KiCad schematic (older format))
At the start: 1 part

Commit message: Update dokumentasi 07112019
Other:
- note added: "MotorKonektor - Wire - DB25 \n+5V : 1 - Merah - 19\nS : 2 - Biru - 7\nGND : 4 - Hitam - 20"
- note removed: "MotorKonektor - Wire - DB25 \n+5V : 1 - Merah - 20\nS : 2 - Biru - 8\nGND : 4 - Hitam - 21"
Changed lines of the file:
@@
 MotorKonektor
 Text Notes 2550 4950 0    60   ~ 0
-MotorKonektor - Wire - DB25 \n+5V : 1 - Merah - 20\nS : 2 - Biru - 8\nGND : 4 - Hitam - 21
+MotorKonektor - Wire - DB25 \n+5V : 1 - Merah - 19\nS : 2 - Biru - 7\nGND : 4 - Hitam - 20
 $EndSCHEMATC
