File: circuit/file5D586D56.sch (KiCad schematic (older format))
At the start: 16 parts, among them J1 Encoder_Conn, J2 Conn_01x03_Female, SW1 SW_Push_45deg, SW2 SW_Push_45deg, SW3 SW_Push_45deg, U2 LM324

Commit message: Update dokumentasi 07112019
Parts:
- added J? (x3): Encoder_Conn, symbol Conn_01x04_Female
- added R? (x4): R, symbol R
- added RV? (x4): POT_TRIM, symbol POT_TRIM
- added U? (x4): LM324, symbol LM324
Connections:
- net Encoder_Dir is gone; now on net ENCODER_IN_Tick: J1.3 (Pin_3), J?.2, U2.5 (+)
- net Encoder_Tick is gone; now on net ENCODER_IN_Tick: J1.2 (Pin_2), J?.14 (P14), U2.3 (+)
- net +5V: now also J?.19 (P19), J?.1 (Pin_1), J?.1 (Pin_1), J?.1 (Pin_1), R?.1, R?.1, R?.1, R?.1, RV?.1, RV?.1, RV?.1, RV?.1, U?.4 (V+), U?.4 (V+), U?.4 (V+), U?.4 (V+); no longer J?.20 (P20)
- net -VDC: now also J?.20 (P20), J?.4 (Pin_4), J?.4 (Pin_4), RV?.3, RV?.3, RV?.3, RV?.3, U?.11 (V-), U?.11 (V-), U?.11 (V-), U?.11 (V-); no longer J?.21 (P21)
- net ENCODER_IN_Dir: now also U?.1, U?.1, U?.2 (-), U?.2 (-)
- net ENCODER_IN_Tick: now also J?.2 (Pin_2), J?.2 (Pin_2), J?.2 (Pin_2), J?.3 (Pin_3), J?.3 (Pin_3), J?.3 (Pin_3), R?.2, R?.2, R?.2, R?.2, U?.1, U?.1, U?.2 (-), U?.2 (-), U?.3 (+), U?.3 (+), U?.3 (+), U?.3 (+)
- net PositionTrigger: now also J?.7; no longer J?.8
