File: circuit/GoWinElectricalv2/GowinController.sch (KiCad schematic (older format))
At the start: 20 parts, among them Q1 IRF3205, U1 LM324, U2 HCPL3120

Commit message: Update dokumentasi 07112019
Parts:
- removed C1: CP, Capacitors_THT:CP_Radial_D12.5mm_P5.00mm, symbol CP
- removed U2: HCPL3120, Housings_DIP:DIP-8_W7.62mm, symbol HCPL3120
- added R? (x4): 10k, symbol R
- added RV? (x7): POT_TRIM, Potentiometers:Potentiometer_Trimmer_Bourns_3296W, symbol POT_TRIM
- added U? (x5): LM324, Housings_DIP:DIP-14_W7.62mm_Socket_LongPads, symbol LM324
Connections:
- net Encoder_Dir is gone; now on net ENCODER_IN_Dir: Encoder1.3 (Pin_3), U1.5 (+)
- net Encoder_Tick is gone; now on net ENCODER_IN_Tick: Encoder1.2 (Pin_2), U1.3 (+)
- net +5V: now also R?.1, R?.1, R?.1, R?.1, RV?.1, RV?.1, RV?.1, RV?.1, RV?.1, RV?.1, RV?.1, U?.4 (V+), U?.4 (V+), U?.4 (V+), U?.4 (V+), U?.4 (V+)
- net ENCODER_IN_Dir: now also R?.2, R?.2, U?.1, U?.1, U?.2 (-), U?.2 (-), U?.3 (+), U?.3 (+)
- net ENCODER_IN_Tick: now also R?.2, R?.2, U?.1, U?.1, U?.2 (-), U?.2 (-), U?.3 (+), U?.3 (+)
- net GND: now also R2.1, RV?.3, RV?.3, RV?.3, RV?.3, RV?.3, RV?.3, RV?.3, U?.11 (V-), U?.11 (V-), U?.11 (V-), U?.11 (V-), U?.11 (V-)
- net PositionTrigger: now also U?.3 (+)
- net PositionTrigger_IN: now also U?.1, U?.2 (-)
- net at R2.2: now also Q1.1 (G)
Other:
- moved on the sheet: R1, R2
