File: circuit/GoWinElectricalv2/GowinController.sch (KiCad schematic (older format))
At the start: 34 parts, among them Q1 IRF3205, U1 LM324

Commit message: Update 11_11_2019
Parts:
- removed RV1, RV2: POT_TRIM, Potentiometers:Potentiometer_Trimmer_Bourns_3296W, symbol POT_TRIM
- removed unit 2 of U1
- removed unit 1 of U1
Other:
- moved on the sheet: BatterySupply1, D1, DCDCConverter1, DashboardConn1, Encoder1, MotorConn1, PinHeadBawah1, PinHeadKanan1, PinHeadKiri1, PositionTrigger1, Q1, R1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
