File: circuit/GoWinElectricalv2/_autosave-GoWinElectricalv2.kicad_pcb (KiCad board)
At the start: 4 copper layers, 35.6 x 96.5 mm, 23 parts, among them Q1 IRF3205, U1 LM324, U2 HCPL3120

Commit message: Update dokumentasi 07112019
Other:
- board text added: "+VDC"
- board text added: "BAT+"
- board text added: "BAT-"
- board text added: "EncoderDir_Pot"
- board text added: "EncoderTick_Pot"
- board text added: "MOTOR+"
- board text added: "MOTOR-"
- board text added: "PositionTrigger"
- board text added: "PositionTrigger_GND"
- board text added: "PositionTrigger_Pot"
Changed lines of the file:
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@@
     (links 100)
     (no_connects 17)
-    (area 132.004999 64.948999 167.715001 161.619001)
+    (area 120.769333 45.149714 177.803143 161.897)
     (thickness 1.6)
-    (drawings 18)
+    (drawings 28)
     (tracks 306)
     (zones 0)
@@
     (pad_to_mask_clearance 0.2)
     (aux_axis_origin 0 0)
-    (visible_elements 7FFFFFFF)
+    (visible_elements 7FFCFFF7)
     (pcbplotparams
       (layerselection 0x00030_80000001)
@@
     (pad 1 thru_hole circle (at 0 0) (size 5.7 5.7) (drill 3.2) (layers *.Cu *.Mask))
   )
+  (gr_text "PositionTrigger_Pot\n" (at 123.1265 131.953) (layer F.Adhes)
+    (effects (font (size 1.5 1.5) (thickness 0.3)))
+  )
+  (gr_text "EncoderTick_Pot\n" (at 122.6185 122.301) (layer F.Adhes)
+    (effects (font (size 1.5 1.5) (thickness 0.3)))
+  )
+  (gr_text "EncoderDir_Pot\n" (at 122.682 112.268) (layer F.Adhes)
+    (effects (font (size 1.5 1.5) (thickness 0.3)))
+  )
+  (gr_text BAT- (at 168.402 143.764) (layer In1.Cu)
+    (effects (font (size 1.5 1.5) (thickness 0.3)))
+  )
+  (gr_text BAT+ (at 168.402 141.224) (layer In1.Cu)
+    (effects (font (size 1.5 1.5) (thickness 0.3)))
+  )
+  (gr_text MOTOR+ (at 170.434 137.16) (layer In1.Cu)
+    (effects (font (size 1.5 1.5) (thickness 0.3)))
+  )
+  (gr_text MOTOR- (at 170.434 134.62) (layer In1.Cu)
+    (effects (font (size 1.5 1.5) (thickness 0.3)))
+  )
+  (gr_text +VDC (at 142.494 134.62 90) (layer In1.Cu)
+    (effects (font (size 1.5 1.5) (thickness 0.3)))
+  )
+  (gr_text PositionTrigger (at 147.32 139.7 90) (layer In1.Cu)
+    (effects (font (size 1.5 1.5) (thickness 0.3)))
+  )
+  (gr_text PositionTrigger_GND (at 150.114 142.24 90) (layer In1.Cu)
+    (effects (font (size 1.5 1.5) (thickness 0.3)))
+  )
   (gr_text GND (at 166.878 124.46) (layer In1.Cu)
