File: circuit/GoWinElectricalv2/_saved_GowinController.sch (KiCad schematic (older format))
At the start: 34 parts, among them Q1 IRF3205, U1 LM324

Commit message: Update dokumentasi 07112019
Connections:
- net at Q1.1 (G), R2.2: now also R1.1
Other:
- moved on the sheet: RV?, U?A
Changed lines of the file:
@@
 L LM324 U?
 U 1 1 5DC20097
-P 25600 7200
-F 0 "U?" H 25600 7400 50  0000 L CNN
-F 1 "LM324" H 25600 7000 50  0000 L CNN
-F 2 "Housings_DIP:DIP-14_W7.62mm_Socket_LongPads" H 25550 7300 50  0001 C CNN
-F 3 "" H 25650 7400 50  0001 C CNN
-	1    25600 7200
+P 18600 6250
+F 0 "U?" H 18600 6450 50  0000 L CNN
+F 1 "LM324" H 18600 6050 50  0000 L CNN
+F 2 "Housings_DIP:DIP-14_W7.62mm_Socket_LongPads" H 18550 6350 50  0001 C CNN
+F 3 "" H 18650 6450 50  0001 C CNN
+	1    18600 6250
 	1    0    0    -1
 $EndComp
@@
 L POT_TRIM RV?
 U 1 1 5DC2009D
-P 24800 7300
-F 0 "RV?" V 24625 7300 50  0000 C CNN
-F 1 "POT_TRIM" V 24700 7300 50  0000 C CNN
-F 2 "Potentiometers:Potentiometer_Trimmer_Bourns_3296W" H 24800 7300 50  0001 C CNN
-F 3 "" H 24800 7300 50  0001 C CNN
-	1    24800 7300
+P 17800 6350
+F 0 "RV?" V 17625 6350 50  0000 C CNN
+F 1 "POT_TRIM" V 17700 6350 50  0000 C CNN
+F 2 "Potentiometers:Potentiometer_Trimmer_Bourns_3296W" H 17800 6350 50  0001 C CNN
+F 3 "" H 17800 6350 50  0001 C CNN
+	1    17800 6350
 	1    0    0    -1
 $EndComp
@@
 L +5V #PWR?
 U 1 1 5DC200A3
-P 24800 6900
-F 0 "#PWR?" H 24800 6750 50  0001 C CNN
-F 1 "+5V" H 24800 7040 50  0000 C CNN
-F 2 "" H 24800 6900 50  0001 C CNN
-F 3 "" H 24800 6900 50  0001 C CNN
-	1    24800 6900
+P 17800 5950
+F 0 "#PWR?" H 17800 5800 50  0001 C CNN
+F 1 "+5V" H 17800 6090 50  0000 C CNN
+F 2 "" H 17800 5950 50  0001 C CNN
+F 3 "" H 17800 5950 50  0001 C CNN
+	1    17800 5950
 	1    0    0    -1
 $EndComp
@@
 L +5V #PWR?
 U 1 1 5DC200A9
-P 25500 6800
-F 0 "#PWR?" H 25500 6650 50  0001 C CNN
-F 1 "+5V" H 25500 6940 50  0000 C CNN
-F 2 "" H 25500 6800 50  0001 C CNN
-F 3 "" H 25500 6800 50  0001 C CNN
-	1    25500 6800
+P 18500 5850
+F 0 "#PWR?" H 18500 5700 50  0001 C CNN
+F 1 "+5V" H 18500 5990 50  0000 C CNN
+F 2 "" H 18500 5850 50  0001 C CNN
+F 3 "" H 18500 5850 50  0001 C CNN
+	1    18500 5850
 	1    0    0    -1
 $EndComp
@@
 L GND #PWR?
 U 1 1 5DC200AF
-P 25500 7600
-F 0 "#PWR?" H 25500 7350 50  0001 C CNN
-F 1 "GND" H 25500 7450 50  0000 C CNN
-F 2 "" H 25500 7600 50  0001 C CNN
-F 3 "" H 25500 7600 50  0001 C CNN
-	1    25500 7600
+P 18500 6650
+F 0 "#PWR?" H 18500 6400 50  0001 C CNN
+F 1 "GND" H 18500 6500 50  0000 C CNN
+F 2 "" H 18500 6650 50  0001 C CNN
+F 3 "" H 18500 6650 50  0001 C CNN
+	1    18500 6650
 	1    0    0    -1
 $EndComp
@@
 L GND #PWR?
 U 1 1 5DC200B5
-P 24800 7600
-F 0 "#PWR?" H 24800 7350 50  0001 C CNN
-F 1 "GND" H 24800 7450 50  0000 C CNN
-F 2 "" H 24800 7600 50  0001 C CNN
-F 3 "" H 24800 7600 50  0001 C CNN
-	1    24800 7600
+P 17800 6650
+F 0 "#PWR?" H 17800 6400 50  0001 C CNN
+F 1 "GND" H 17800 6500 50  0000 C CNN
+F 2 "" H 17800 6650 50  0001 C CNN
+F 3 "" H 17800 6650 50  0001 C CNN
+	1    17800 6650
 	1    0    0    -1
 $EndComp
-Text HLabel 24600 7100 0    60   Input ~ 0
+Text HLabel 17600 6150 0    60   Input ~ 0
 PositionTrigger
-Text HLabel 26000 7200 2    60   Input ~ 0
+Text HLabel 19000 6250 2    60   Input ~ 0
 PositionTrigger_IN
 Wire Wire Line
@@
 Connection ~ 7500 4450
 Wire Wire Line
-	7350 5350 7500 5350
+	7150 5350 7500 5350
 Wire Wire Line
 	7800 5550 7800 6050
@@
 	14850 5750 14850 5700
 Wire Wire Line
-	25900 7200 26000 7200
-Wire Wire Line
-	24800 7450 24800 7600
-Wire Wire Line
-	25500 7500 25500 7600
-Wire Wire Line
-	25500 6800 25500 6900
-Wire Wire Line
-	24800 6900 24800 7150
-Wire Wire Line
-	24600 7100 25300 7100
-Wire Wire Line
-	25300 7300 25100 7300
-Wire Wire Line
-	25100 7300 25100 6850
-Wire Wire Line
-	25100 6850 25950 6850
-Wire Wire Line
-	25950 6850 25950 7200
-Connection ~ 25950 7200
+	18900 6250 19000 6250
+Wire Wire Line
+	17800 6500 17800 6650
+Wire Wire Line
+	18500 6550 18500 6650
+Wire Wire Line
+	18500 5850 18500 5950
+Wire Wire Line
+	17800 5950 17800 6200
+Wire Wire Line
+	17600 6150 18300 6150
+Wire Wire Line
+	18300 6350 18100 6350
+Wire Wire Line
+	18100 6350 18100 5900
+Wire Wire Line
+	18100 5900 18950 5900
+Wire Wire Line
+	18950 5900 18950 6250
+Connection ~ 18950 6250
 Wire Wire Line
 	7350 5450 7350 5450
@@
 Wire Wire Line
 	7350 5750 7800 5750
+Connection ~ 7350 5350
 $EndSCHEMATC
